File: PCB/PCB_Test/PCB_Test.kicad_sch (KiCad schematic)
At the start: 2 parts, among them U1 ESP32-WROOM-32E, U2 LM317_SOT-223

Commit message: update
Parts:
- removed U1: ESP32-WROOM-32E, RF_Module:ESP32-WROOM-32D, symbol RF_Module:ESP32-WROOM-32E
- removed U2: LM317_SOT-223, Package_TO_SOT_SMD:SOT-223-3_TabPin2, symbol Regulator_Linear:LM317_SOT-223
- added U1: ~, ESP32-footprints-Lib:ESP32DEVKITV1, symbol ESP32_DEVKITV1:ESP32_DEVKITV1
Changed lines of the file:
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@@
 	(paper "A4")
 	(symbol
-		(lib_id "Regulator_Linear:LM317_SOT-223")
-		(at 66.04 67.31 0)
+		(lib_id "ESP32_DEVKITV1:ESP32_DEVKITV1")
+		(at 90.17 68.58 0)
 		(unit 1)
 		(exclude_from_sim no)
@@
 		(dnp no)
 		(fields_autoplaced yes)
-		(property "Reference" "U2"
-			(at 66.04 60.96 0)
+		(property "Reference" "U1"
+			(at 90.805 41.91 0)
 			(effects
 				(font
@@
 			)
 		)
-		(property "Value" "LM317_SOT-223"
-			(at 66.04 63.5 0)
+		(property "Value" "~"
+			(at 90.805 44.45 0)
 			(effects
 				(font
@@
 			)
 		)
-		(property "Footprint" "Package_TO_SOT_SMD:SOT-223-3_TabPin2"
-			(at 66.04 60.96 0)
-			(effects
-				(font
-					(size 1.27 1.27)
-					(italic yes)
-				)
-				(hide yes)
-			)
-		)
-		(property "Datasheet" "http://www.ti.com/lit/ds/symlink/lm317.pdf"
-			(at 66.04 67.31 0)
+		(property "Footprint" "ESP32-footprints-Lib:ESP32DEVKITV1"
+			(at 90.17 68.58 0)
 			(effects
 				(font
@@
 			)
 		)
-		(property "Description" "1.5A 35V Adjustable Linear Regulator, SOT-223"
-			(at 66.04 67.31 0)
+		(property "Datasheet" ""
+			(at 90.17 68.58 0)
 			(effects
 				(font
@@
 			)
 		)
-		(pin "3"
-		)
-		(pin "2"
-		)
-		(pin "1"
-		)
-		(instances
-			(project ""
-				(path "/271f5698-945e-4905-aaf5-70f20bf42c62"
-					(reference "U2")
-					(unit 1)
-				)
-			)
-		)
-	)
-	(symbol
-		(lib_id "RF_Module:ESP32-WROOM-32E")
-		(at 119.38 85.09 0)
-		(unit 1)
-		(exclude_from_sim no)
-		(in_bom yes)
-		(on_board yes)
-		(dnp no)
-		(fields_autoplaced yes)
-		(property "Reference" "U1"
-			(at 121.5233 46.99 0)
-			(effects
-				(font
-					(size 1.27 1.27)
-				)
-				(justify left)
-			)
-		)
-		(property "Value" "ESP32-WROOM-32E"
-			(at 121.5233 49.53 0)
-			(effects
-				(font
-					(size 1.27 1.27)
-				)
-				(justify left)
-			)
-		)
-		(property "Footprint" "RF_Module:ESP32-WROOM-32D"
-			(at 135.89 119.38 0)
+		(property "Description" ""
+			(at 90.17 68.58 0)
 			(effects
 				(font
@@
 			)
 		)
-		(property "Datasheet" "https://www.espressif.com/sites/default/files/documentation/esp32-wroom-32e_esp32-wroom-32ue_datasheet_en.pdf"
-			(at 119.38 85.09 0)
-			(effects
-				(font
-					(size 1.27 1.27)
-				)
-				(hide yes)
-			)
+		(pin "2"
 		)
-		(property "Description" "RF Module, ESP32-D0WD-V3 SoC, without PSRAM, Wi-Fi 802.11b/g/n, Bluetooth, BLE, 32-bit, 2.7-3.6V, onboard antenna, SMD"
-			(at 119.38 85.09 0)
-			(effects
-				(font
-					(size 1.27 1.27)
-				)
-				(hide yes)
-			)
+		(pin "1"
 		)
-		(pin "34"
+		(pin "8"
+		)
+		(pin "16"
+		)
+		(pin "12"
+		)
+		(pin "15"
+		)
+		(pin "30"
+		)
+		(pin "26"
+		)
+		(pin "25"
+		)
+		(pin "3"
+		)
+		(pin "6"
+		)
+		(pin "14"
+		)
+		(pin "4"
+		)
+		(pin "9"
+		)
+		(pin "17"
+		)
+		(pin "28"
+		)
+		(pin "5"
+		)
+		(pin "7"
+		)
+		(pin "10"
+		)
+		(pin "11"
+		)
+		(pin "13"
 		)
 		(pin "29"
 		)
-		(pin "26"
-		)
 		(pin "27"
-		)
-		(pin "35"
-		)
-		(pin "15"
-		)
-		(pin "19"
-		)
-		(pin "4"
-		)
-		(pin "31"
-		)
-		(pin "18"
-		)
-		(pin "39"
 		)
 		(pin "20"
 		)
-		(pin "5"
-		)
-		(pin "3"
-		)
-		(pin "2"
-		)
-		(pin "38"
-		)
-		(pin "1"
-		)
-		(pin "17"
-		)
-		(pin "25"
-		)
-		(pin "22"
-		)
-		(pin "32"
+		(pin "18"
 		)
 		(pin "21"
@@
 		(pin "24"
 		)
-		(pin "14"
-		)
-		(pin "16"
-		)
-		(pin "13"
+		(pin "19"
 		)
 		(pin "23"
 		)
-		(pin "30"
-		)
-		(pin "12"
-		)
-		(pin "28"
-		)
-		(pin "37"
-		)
-		(pin "11"
-		)
-		(pin "33"
-		)
-		(pin "8"
-		)
-		(pin "7"
-		)
-		(pin "36"
-		)
-		(pin "6"
-		)
-		(pin "9"
-		)
-		(pin "10"
+		(pin "22"
 		)
 		(instances
